File: PCB/Rev1/PH60Slim-Choc.kicad_sch (KiCad schematic)
At the start: 36 parts, among them J1 USB_C_Receptacle_USB2.0_16P, J2 Conn_01x02, U2 W25Q128JVS, U3 RP2040, U4 XC6206PxxxMR, Y1 Crystal_GND24

Commit message: Fuse and silkscreen update.
Parts:
- F1: value 500ma -> 750ma; footprint Fuse:Fuse_0603_1608Metric -> Fuse:Fuse_0805_2012Metric
Changed lines of the file:
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@@
 			)
 		)
-		(property "Value" "500ma"
+		(property "Value" "750ma"
 			(at 73.66 193.04 90)
 			(effects
@@
 			)
 		)
-		(property "Footprint" "Fuse:Fuse_0603_1608Metric"
+		(property "Footprint" "Fuse:Fuse_0805_2012Metric"
 			(at 78.74 195.58 0)
 			(effects
@@
 		)
 		(instances
-			(project "PH60_Rev2"
+			(project "PH60Slim-Choc"
 				(path "/dca0f898-8fdb-4522-a51d-f4f4238906e7"
 					(page "3")
@@
 		)
 		(instances
-			(project "PH60_Rev2"
+			(project "PH60Slim-Choc"
 				(path "/dca0f898-8fdb-4522-a51d-f4f4238906e7"
 					(page "2")
